File: cob_panel_mini/cob_panel_mini.sch (KiCad schematic (older format))
At the start: 25 parts, among them J1 Conn_01x03, J2 Conn_01x03, Q1 Q_NPN_BEC, Q2 Q_NPN_BEC, Q3 Q_NPN_BEC, U1 MOSFET_N_SI3424CDV-T1-GE3, U2 WS2811, U3 MOSFET_N_SI3424CDV-T1-GE3, U4 MOSFET_N_SI3424CDV-T1-GE3, U5 3_Inverter_TC7WH14FU,LJ(CT

Commit message: WIP associate footprints
Parts:
- added C4: 10uF, Capacitor_SMD:C_0805_2012Metric, symbol Device:C
- C1: footprint (none) -> Capacitor_SMD:C_0805_2012Metric
- C2, C3: footprint (none) -> Capacitor_SMD:C_0603_1608Metric
- D1: footprint (none) -> LED_SMD:LED_RGB_Getian_GT-P6PRGB4303
- J1, J2: footprint (none) -> Connector_PinHeader_2.54mm:PinHeader_1x03_P2.54mm_Vertical
- Q1, Q2, Q3: footprint (none) -> Package_TO_SOT_SMD:SOT-23
- R1, R10, R11, R3, R4, R5, R7, R9: footprint (none) -> Resistor_SMD:R_0603_1608Metric
- R2, R6, R8: footprint (none) -> Resistor_SMD:R_0805_2012Metric_Pad1.15x1.40mm_HandSolder
- U1: footprint (none) -> homebrew:6-TSOP-MOSFET-SI3424CDV-T1-GE3
- U2: renamed from U3; footprint (none) -> homebrew:6-TSOP-MOSFET-SI3424CDV-T1-GE3
- U3: renamed from U4; footprint (none) -> homebrew:6-TSOP-MOSFET-SI3424CDV-T1-GE3
- U4: renamed from U2; footprint (none) -> Package_SO:SOP-8_3.76x4.96mm_P1.27mm
- U5: footprint (none) -> Package_SO:TSSOP-8_3x3mm_P0.65mm
Connections:
- net GND: now also C4.2
- net VCC: now also C4.1
Changed lines of the file:
@@
 F 0 "J1" H 768 975 50  0000 C CNN
 F 1 "Conn_01x03" H 768 1066 50  0000 C CNN
-F 2 "" H 850 1300 50  0001 C CNN
+F 2 "Connector_PinHeader_2.54mm:PinHeader_1x03_P2.54mm_Vertical" H 850 1300 50  0001 C CNN
 F 3 "~" H 850 1300 50  0001 C CNN
 	1    850  1300
@@
 F 0 "C1" H 1215 3446 50  0000 L CNN
 F 1 "10uF" H 1215 3355 50  0000 L CNN
-F 2 "" H 1138 3250 50  0001 C CNN
+F 2 "Capacitor_SMD:C_0805_2012Metric" H 1138 3250 50  0001 C CNN
 F 3 "~" H 1100 3400 50  0001 C CNN
 	1    1100 3400
@@
 Connection ~ 1100 1450
 $Comp
-L Driver_LED:WS2811 U2
+L Driver_LED:WS2811 U4
 U 1 1 5DB3C45F
 P 3600 1350
-F 0 "U2" H 3300 1650 50  0000 C CNN
+F 0 "U4" H 3300 1650 50  0000 C CNN
 F 1 "WS2811" H 3250 1750 50  0000 C CNN
-F 2 "" H 3300 1500 50  0001 C CNN
+F 2 "Package_SO:SOP-8_3.76x4.96mm_P1.27mm" H 3300 1500 50  0001 C CNN
 F 3 "https://cdn-shop.adafruit.com/datasheets/WS2811.pdf" H 3400 1600 50  0001 C CNN
 	1    3600 1350
@@
 F 0 "R5" H 3670 946 50  0000 L CNN
 F 1 "33" H 3670 855 50  0000 L CNN
-F 2 "" V 3530 900 50  0001 C CNN
+F 2 "Resistor_SMD:R_0603_1608Metric" V 3530 900 50  0001 C CNN
 F 3 "~" H 3600 900 50  0001 C CNN
 	1    3600 900
@@
 F 0 "C2" H 4815 1296 50  0000 L CNN
 F 1 ".1uF" H 4815 1205 50  0000 L CNN
-F 2 "" H 4738 1100 50  0001 C CNN
+F 2 "Capacitor_SMD:C_0603_1608Metric" H 4738 1100 50  0001 C CNN
 F 3 "~" H 4700 1250 50  0001 C CNN
 	1    4700 1250
@@
 F 0 "R3" V 2843 1250 50  0000 C CNN
 F 1 "33" V 2934 1250 50  0000 C CNN
-F 2 "" V 2980 1250 50  0001 C CNN
+F 2 "Resistor_SMD:R_0603_1608Metric" V 2980 1250 50  0001 C CNN
 F 3 "~" H 3050 1250 50  0001 C CNN
 	1    3050 1250
@@
 F 0 "U5" H 9400 2000 50  0000 C CNN
 F 1 "3_Inverter_TC7WH14FU,LJ(CT" H 9900 1350 50  0000 C CNN
-F 2 "" H 9150 1700 50  0001 C CNN
+F 2 "Package_SO:TSSOP-8_3x3mm_P0.65mm" H 9150 1700 50  0001 C CNN
 F 3 "" H 9150 1700 50  0001 C CNN
 	1    9250 1700
@@
 F 0 "C3" H 9765 1146 50  0000 L CNN
 F 1 ".1uF" H 9765 1055 50  0000 L CNN
-F 2 "" H 9688 950 50  0001 C CNN
+F 2 "Capacitor_SMD:C_0603_1608Metric" H 9688 950 50  0001 C CNN
 F 3 "~" H 9650 1100 50  0001 C CNN
 	1    9650 1100
@@
 F 0 "R11" H 8820 1446 50  0000 L CNN
 F 1 "1k" H 8820 1355 50  0000 L CNN
-F 2 "" V 8680 1400 50  0001 C CNN
+F 2 "Resistor_SMD:R_0603_1608Metric" V 8680 1400 50  0001 C CNN
 F 3 "~" H 8750 1400 50  0001 C CNN
 	1    8750 1400
@@
 F 0 "R10" H 8320 1546 50  0000 L CNN
 F 1 "1k" H 8320 1455 50  0000 L CNN
-F 2 "" V 8180 1500 50  0001 C CNN
+F 2 "Resistor_SMD:R_0603_1608Metric" V 8180 1500 50  0001 C CNN
 F 3 "~" H 8250 1500 50  0001 C CNN
 	1    8250 1500
@@
 F 0 "R9" H 7820 1646 50  0000 L CNN
 F 1 "1k" H 7820 1555 50  0000 L CNN
-F 2 "" V 7680 1600 50  0001 C CNN
+F 2 "Resistor_SMD:R_0603_1608Metric" V 7680 1600 50  0001 C CNN
 F 3 "~" H 7750 1600 50  0001 C CNN
 	1    7750 1600
@@
 F 0 "J2" H 6418 975 50  0000 C CNN
 F 1 "Conn_01x03" H 6700 1500 50  0000 C CNN
-F 2 "" H 6500 1300 50  0001 C CNN
+F 2 "Connector_PinHeader_2.54mm:PinHeader_1x03_P2.54mm_Vertical" H 6500 1300 50  0001 C CNN
 F 3 "~" H 6500 1300 50  0001 C CNN
 	1    6500 1300
@@
 F 0 "U1" V 4555 3221 60  0000 R CNN
 F 1 "MOSFET_N_SI3424CDV-T1-GE3" V 4800 4800 60  0000 R CNN
-F 2 "" H 4550 3150 60  0000 C CNN
+F 2 "homebrew:6-TSOP-MOSFET-SI3424CDV-T1-GE3" H 4550 3150 60  0001 C CNN
 F 3 "" H 4550 3150 60  0000 C CNN
 	1    4550 3200
@@
 F 0 "Q1" H 4091 3496 50  0000 L CNN
 F 1 "Q_NPN_BEC" H 4091 3405 50  0000 L CNN
-F 2 "" H 4100 3550 50  0001 C CNN
+F 2 "Package_TO_SOT_SMD:SOT-23" H 4100 3550 50  0001 C CNN
 F 3 "~" H 3900 3450 50  0001 C CNN
 	1    3900 3450
@@
 F 0 "D1" H 1750 2783 50  0000 C CNN
 F 1 "LED_RGB" H 1750 2874 50  0000 C CNN
-F 2 "" H 1750 3200 50  0001 C CNN
+F 2 "LED_SMD:LED_RGB_Getian_GT-P6PRGB4303" H 1750 3200 50  0001 C CNN
 F 3 "~" H 1750 3200 50  0001 C CNN
 	1    1750 3250
@@
 	1050 3250 1100 3250
 Wire Wire Line
-	1200 1150 1750 1150
+	1200 1150 1650 1150
 Wire Wire Line
 	1100 3250 1500 3250
@@
 F 0 "R2" H 4520 3696 50  0000 L CNN
 F 1 ".36" H 4520 3605 50  0000 L CNN
-F 2 "" V 4380 3650 50  0001 C CNN
+F 2 "Resistor_SMD:R_0805_2012Metric_Pad1.15x1.40mm_HandSolder" V 4380 3650 50  0001 C CNN
 F 3 "~" H 4450 3650 50  0001 C CNN
 	1    4450 3650
@@
 F 0 "R1" V 3443 3250 50  0000 C CNN
 F 1 "100" V 3534 3250 50  0000 C CNN
-F 2 "" V 3580 3250 50  0001 C CNN
+F 2 "Resistor_SMD:R_0603_1608Metric" V 3580 3250 50  0001 C CNN
 F 3 "~" H 3650 3250 50  0001 C CNN
 	1    3650 3250
@@
 R_SIGNAL
 $Comp
-L Homebrew:MOSFET_N_SI3424CDV-T1-GE3 U3
+L Homebrew:MOSFET_N_SI3424CDV-T1-GE3 U2
 U 1 1 5DB85194
 P 6500 3200
-F 0 "U3" V 6505 3221 60  0000 R CNN
+F 0 "U2" V 6505 3221 60  0000 R CNN
 F 1 "MOSFET_N_SI3424CDV-T1-GE3" V 6750 4800 60  0000 R CNN
-F 2 "" H 6500 3150 60  0000 C CNN
+F 2 "homebrew:6-TSOP-MOSFET-SI3424CDV-T1-GE3" H 6500 3150 60  0001 C CNN
 F 3 "" H 6500 3150 60  0000 C CNN
 	1    6500 3200
@@
 F 0 "Q2" H 6041 3496 50  0000 L CNN
 F 1 "Q_NPN_BEC" H 6041 3405 50  0000 L CNN
-F 2 "" H 6050 3550 50  0001 C CNN
+F 2 "Package_TO_SOT_SMD:SOT-23" H 6050 3550 50  0001 C CNN
 F 3 "~" H 5850 3450 50  0001 C CNN
 	1    5850 3450
@@
 F 0 "R6" H 6470 3696 50  0000 L CNN
 F 1 ".36" H 6470 3605 50  0000 L CNN
-F 2 "" V 6330 3650 50  0001 C CNN
+F 2 "Resistor_SMD:R_0805_2012Metric_Pad1.15x1.40mm_HandSolder" V 6330 3650 50  0001 C CNN
 F 3 "~" H 6400 3650 50  0001 C CNN
 	1    6400 3650
@@
 F 0 "R4" V 5393 3250 50  0000 C CNN
 F 1 "100" V 5484 3250 50  0000 C CNN
-F 2 "" V 5530 3250 50  0001 C CNN
+F 2 "Resistor_SMD:R_0603_1608Metric" V 5530 3250 50  0001 C CNN
 F 3 "~" H 5600 3250 50  0001 C CNN
 	1    5600 3250
@@
 G_SIGNAL
 $Comp
-L Homebrew:MOSFET_N_SI3424CDV-T1-GE3 U4
+L Homebrew:MOSFET_N_SI3424CDV-T1-GE3 U3
 U 1 1 5DB86559
 P 8450 3200
-F 0 "U4" V 8455 3221 60  0000 R CNN
+F 0 "U3" V 8455 3221 60  0000 R CNN
 F 1 "MOSFET_N_SI3424CDV-T1-GE3" V 8700 4800 60  0000 R CNN
-F 2 "" H 8450 3150 60  0000 C CNN
+F 2 "homebrew:6-TSOP-MOSFET-SI3424CDV-T1-GE3" H 8450 3150 60  0001 C CNN
 F 3 "" H 8450 3150 60  0000 C CNN
 	1    8450 3200
@@
 F 0 "Q3" H 7991 3496 50  0000 L CNN
 F 1 "Q_NPN_BEC" H 7991 3405 50  0000 L CNN
-F 2 "" H 8000 3550 50  0001 C CNN
+F 2 "Package_TO_SOT_SMD:SOT-23" H 8000 3550 50  0001 C CNN
 F 3 "~" H 7800 3450 50  0001 C CNN
 	1    7800 3450
@@
 F 0 "R8" H 8420 3696 50  0000 L CNN
 F 1 ".36" H 8420 3605 50  0000 L CNN
-F 2 "" V 8280 3650 50  0001 C CNN
+F 2 "Resistor_SMD:R_0805_2012Metric_Pad1.15x1.40mm_HandSolder" V 8280 3650 50  0001 C CNN
 F 3 "~" H 8350 3650 50  0001 C CNN
 	1    8350 3650
@@
 F 0 "R7" V 7343 3250 50  0000 C CNN
 F 1 "100" V 7434 3250 50  0000 C CNN
-F 2 "" V 7480 3250 50  0001 C CNN
+F 2 "Resistor_SMD:R_0603_1608Metric" V 7480 3250 50  0001 C CNN
 F 3 "~" H 7550 3250 50  0001 C CNN
 	1    7550 3250
@@
 Text GLabel 7400 3250 0    50   Input ~ 0
 B_SIGNAL
+$Comp
+L Device:C C4
+U 1 1 5DB97820
+P 1650 1300
+F 0 "C4" H 1765 1346 50  0000 L CNN
+F 1 "10uF" H 1765 1255 50  0000 L CNN
+F 2 "Capacitor_SMD:C_0805_2012Metric" H 1688 1150 50  0001 C CNN
+F 3 "~" H 1650 1300 50  0001 C CNN
+	1    1650 1300
+	1    0    0    -1
+$EndComp
+Connection ~ 1650 1150
+Wire Wire Line
+	1650 1150 1750 1150
 $EndSCHEMATC
