File: cob_2x2/cob_2x2.sch (KiCad schematic (older format))
At the start: 18 parts, among them J1 Conn_01x02, J3 Anderson_two_redblack, J4 Conn_01x06_Female, J5 Conn_01x06_Male, U1 5V_REG_AP7370-50W5-7

Commit message: Hardware revision v1.0 complete
Parts:
- removed H6: MountingHole, homebrew:MountingHole_2.7mm_M2.5, symbol Mechanical:MountingHole
- added JP1: Jumper, Connector_PinHeader_2.54mm:PinHeader_1x02_P2.54mm_Vertical, symbol Device:Jumper
- H1, H2, H3, H4, H5: footprint homebrew:MountingHole_2.7mm_M2.5 -> homebrew:HOLE_5MM_#8
Connections:
- net SIGNAL_IN: now also JP1.1; no longer J4.6 (Pin_6)
- new net: J4.6 (Pin_6), JP1.2
Other:
- moved on the sheet: J5
Changed lines of the file:
@@
 F 0 "H1" H 10450 696 50  0000 L CNN
 F 1 "MountingHole" H 10450 605 50  0000 L CNN
-F 2 "homebrew:MountingHole_2.7mm_M2.5" H 10350 650 50  0001 C CNN
+F 2 "homebrew:HOLE_5MM_#8" H 10350 650 50  0001 C CNN
 F 3 "~" H 10350 650 50  0001 C CNN
 	1    10350 650
@@
 F 0 "H2" H 10450 846 50  0000 L CNN
 F 1 "MountingHole" H 10450 755 50  0000 L CNN
-F 2 "homebrew:MountingHole_2.7mm_M2.5" H 10350 800 50  0001 C CNN
+F 2 "homebrew:HOLE_5MM_#8" H 10350 800 50  0001 C CNN
 F 3 "~" H 10350 800 50  0001 C CNN
 	1    10350 800
@@
 F 0 "H3" H 10450 996 50  0000 L CNN
 F 1 "MountingHole" H 10450 905 50  0000 L CNN
-F 2 "homebrew:MountingHole_2.7mm_M2.5" H 10350 950 50  0001 C CNN
+F 2 "homebrew:HOLE_5MM_#8" H 10350 950 50  0001 C CNN
 F 3 "~" H 10350 950 50  0001 C CNN
 	1    10350 950
@@
 F 0 "H4" H 10450 1146 50  0000 L CNN
 F 1 "MountingHole" H 10450 1055 50  0000 L CNN
-F 2 "homebrew:MountingHole_2.7mm_M2.5" H 10350 1100 50  0001 C CNN
+F 2 "homebrew:HOLE_5MM_#8" H 10350 1100 50  0001 C CNN
 F 3 "~" H 10350 1100 50  0001 C CNN
 	1    10350 1100
@@
 	1    0    0    -1
 $EndComp
-$Comp
-L Mechanical:MountingHole H5
-U 1 1 5DF3B8FC
-P 10350 1250
-F 0 "H5" H 10450 1296 50  0000 L CNN
-F 1 "MountingHole" H 10450 1205 50  0000 L CNN
-F 2 "homebrew:MountingHole_2.7mm_M2.5" H 10350 1250 50  0001 C CNN
-F 3 "~" H 10350 1250 50  0001 C CNN
-	1    10350 1250
-	1    0    0    -1
-$EndComp
-$Comp
-L Mechanical:MountingHole H6
-U 1 1 5DF3B902
-P 10350 1400
-F 0 "H6" H 10450 1446 50  0000 L CNN
-F 1 "MountingHole" H 10450 1355 50  0000 L CNN
-F 2 "homebrew:MountingHole_2.7mm_M2.5" H 10350 1400 50  0001 C CNN
-F 3 "~" H 10350 1400 50  0001 C CNN
-	1    10350 1400
-	1    0    0    -1
-$EndComp
 Wire Wire Line
 	4250 4350 4050 4350
@@
 	1700 7050 1700 7100
 NoConn ~ 1550 7200
-Text GLabel 1550 7300 2    50   Input ~ 0
+Text GLabel 2250 7400 2    50   Input ~ 0
 SIGNAL_IN
 Wire Wire Line
 	1700 7050 2150 7050
-Text GLabel 3250 6850 0    50   Input ~ 0
+Text GLabel 4150 6850 0    50   Input ~ 0
 12V_RAW
 $Comp
 L power:GND #PWR06
 U 1 1 5DF2CE82
-P 2850 7050
-F 0 "#PWR06" H 2850 6800 50  0001 C CNN
-F 1 "GND" H 2855 6877 50  0000 C CNN
-F 2 "" H 2850 7050 50  0001 C CNN
-F 3 "" H 2850 7050 50  0001 C CNN
-	1    2850 7050
-	1    0    0    -1
-$EndComp
-Wire Wire Line
-	3500 6800 3350 6800
-Wire Wire Line
-	3350 6800 3350 6850
-Wire Wire Line
-	3350 6900 3500 6900
-Wire Wire Line
-	3500 7000 3350 7000
-Wire Wire Line
-	3350 7000 3350 7050
-Wire Wire Line
-	3350 7100 3500 7100
-Text GLabel 3500 7300 0    50   Input ~ 0
+P 3750 7050
+F 0 "#PWR06" H 3750 6800 50  0001 C CNN
+F 1 "GND" H 3755 6877 50  0000 C CNN
+F 2 "" H 3750 7050 50  0001 C CNN
+F 3 "" H 3750 7050 50  0001 C CNN
+	1    3750 7050
+	1    0    0    -1
+$EndComp
+Wire Wire Line
+	4400 6800 4250 6800
+Wire Wire Line
+	4250 6800 4250 6850
+Wire Wire Line
+	4250 6900 4400 6900
+Wire Wire Line
+	4400 7000 4250 7000
+Wire Wire Line
+	4250 7000 4250 7050
+Wire Wire Line
+	4250 7100 4400 7100
+Text GLabel 4400 7300 0    50   Input ~ 0
 SIGNAL_OUT
 $Comp
 L Connector:Conn_01x06_Male J5
 U 1 1 5DFA4554
-P 3700 7000
-F 0 "J5" H 3672 6974 50  0000 R CNN
-F 1 "Conn_01x06_Male" H 3672 6883 50  0000 R CNN
-F 2 "Connector_PinHeader_2.54mm:PinHeader_1x06_P2.54mm_Horizontal" H 3700 7000 50  0001 C CNN
-F 3 "~" H 3700 7000 50  0001 C CNN
-	1    3700 7000
+P 4600 7000
+F 0 "J5" H 4572 6974 50  0000 R CNN
+F 1 "Conn_01x06_Male" H 4572 6883 50  0000 R CNN
+F 2 "Connector_PinHeader_2.54mm:PinHeader_1x06_P2.54mm_Horizontal" H 4600 7000 50  0001 C CNN
+F 3 "~" H 4600 7000 50  0001 C CNN
+	1    4600 7000
 	-1   0    0    -1
 $EndComp
-NoConn ~ 3500 7200
-Wire Wire Line
-	3250 6850 3350 6850
-Connection ~ 3350 6850
-Wire Wire Line
-	3350 6850 3350 6900
-Wire Wire Line
-	2850 7050 3350 7050
-Connection ~ 3350 7050
-Wire Wire Line
-	3350 7050 3350 7100
+NoConn ~ 4400 7200
+Wire Wire Line
+	4150 6850 4250 6850
+Connection ~ 4250 6850
+Wire Wire Line
+	4250 6850 4250 6900
+Wire Wire Line
+	3750 7050 4250 7050
+Connection ~ 4250 7050
+Wire Wire Line
+	4250 7050 4250 7100
 $Comp
 L Connector_Generic:Conn_01x02 J1
@@
 	-1   0    0    1
 $EndComp
+$Comp
+L Device:Jumper JP1
+U 1 1 5DF9B18A
+P 1950 7400
+F 0 "JP1" H 1950 7650 50  0000 C CNN
+F 1 "Jumper" H 1950 7550 50  0000 C CNN
+F 2 "Connector_PinHeader_2.54mm:PinHeader_1x02_P2.54mm_Vertical" H 1950 7400 50  0001 C CNN
+F 3 "~" H 1950 7400 50  0001 C CNN
+	1    1950 7400
+	-1   0    0    1
+$EndComp
+Wire Wire Line
+	1550 7300 1550 7400
+Wire Wire Line
+	1550 7400 1650 7400
+$Comp
+L Mechanical:MountingHole H5
+U 1 1 5E1404CC
+P 10350 1250
+F 0 "H5" H 10450 1296 50  0000 L CNN
+F 1 "MountingHole" H 10450 1205 50  0000 L CNN
+F 2 "homebrew:HOLE_5MM_#8" H 10350 1250 50  0001 C CNN
+F 3 "~" H 10350 1250 50  0001 C CNN
+	1    10350 1250
+	1    0    0    -1
+$EndComp
 $EndSCHEMATC

Commit message: cob_2x2 v1.1:
- Fix inverter footprint
- Increase size of 5V TVS diode to SOD-523
- Increase clearance for mounting holes by 1mm
- Make mounting holes evenly spaced
Parts:
- removed H5: MountingHole, homebrew:HOLE_5MM_#8, symbol Mechanical:MountingHole
- D10: footprint homebrew:SOD-923 -> Diode_SMD:D_SOD-523
Changed lines of the file:
@@
 F 0 "D10" V 1754 1729 50  0000 L CNN
 F 1 "D_TVS_5V" V 1845 1729 50  0000 L CNN
-F 2 "homebrew:SOD-923" H 1800 1650 50  0001 C CNN
+F 2 "Diode_SMD:D_SOD-523" H 1800 1650 50  0001 C CNN
 F 3 "~" H 1800 1650 50  0001 C CNN
 	1    1800 1650
@@
 Wire Wire Line
 	1550 7400 1650 7400
-$Comp
-L Mechanical:MountingHole H5
-U 1 1 5E1404CC
-P 10350 1250
-F 0 "H5" H 10450 1296 50  0000 L CNN
-F 1 "MountingHole" H 10450 1205 50  0000 L CNN
-F 2 "homebrew:HOLE_5MM_#8" H 10350 1250 50  0001 C CNN
-F 3 "~" H 10350 1250 50  0001 C CNN
-	1    10350 1250
-	1    0    0    -1
-$EndComp
 $EndSCHEMATC
