File: cob_2x2/single_led.sch (KiCad schematic (older format))
At the start: 24 parts, among them U2 AL8860_LED_DRIVER, U3 AL8860_LED_DRIVER, U4 WS2811, U5 AL8860_LED_DRIVER, U6 3_Inverter_TC7WH14FU,LJ(CT

Commit message: Hardware revision v1.0 complete
Parts:
- removed D2: LED_RGB_EP, homebrew:LED_RGB_EPISTAR_6PIN_RGB, symbol Device:LED_RGB_EP
- added D13: LED_RGB, homebrew:LED_RGB_EPISTAR_6PIN_RGB, symbol Device:LED_RGB
Connections:
- no-connect marks 2 -> 1
Changed lines of the file:
@@
 	1    0    0    -1
 $EndComp
-$Comp
-L Device:LED_RGB_EP D?
-U 1 1 5DEA9FB1
-P 1800 3550
-AR Path="/5DEA9FB1" Ref="D?"  Part="1"
-AR Path="/5DE8C448/5DEA9FB1" Ref="D2"  Part="1"
-AR Path="/5DF187B8/5DEA9FB1" Ref="D6"  Part="1"
-AR Path="/5DF1A17B/5DEA9FB1" Ref="D10"  Part="1"
-AR Path="/5DF1A352/5DEA9FB1" Ref="D14"  Part="1"
-AR Path="/5DF1A514/5DEA9FB1" Ref="D18"  Part="1"
-AR Path="/5DF1FB9C/5DEA9FB1" Ref="D22"  Part="1"
-AR Path="/5DF1FDD9/5DEA9FB1" Ref="D26"  Part="1"
-AR Path="/5DF1FFFB/5DEA9FB1" Ref="D30"  Part="1"
-AR Path="/5DF20223/5DEA9FB1" Ref="D34"  Part="1"
-F 0 "D18" H 1800 4047 50  0000 C CNN
-F 1 "LED_RGB_EP" H 1800 3956 50  0000 C CNN
-F 2 "homebrew:LED_RGB_EPISTAR_6PIN_RGB" H 1800 3500 50  0001 C CNN
-F 3 "~" H 1800 3500 50  0001 C CNN
-	1    1800 3550
-	1    0    0    -1
-$EndComp
-NoConn ~ 1800 4050
 Text Label 1700 1750 2    50   ~ 0
 R_SIGNAL
@@
 	1    0    0    -1
 $EndComp
+$Comp
+L Device:LED_RGB D13
+U 1 1 5DFA6EFB
+P 1800 3550
+AR Path="/5DF1A514/5DFA6EFB" Ref="D13"  Part="1"
+AR Path="/5DE8C448/5DFA6EFB" Ref="D2"  Part="1"
+AR Path="/5DF187B8/5DFA6EFB" Ref="D6"  Part="1"
+AR Path="/5DF1FB9C/5DFA6EFB" Ref="D12"  Part="1"
+F 0 "D13" H 1800 4047 50  0000 C CNN
+F 1 "LED_RGB" H 1800 3956 50  0000 C CNN
+F 2 "homebrew:LED_RGB_EPISTAR_6PIN_RGB" H 1800 3500 50  0001 C CNN
+F 3 "~" H 1800 3500 50  0001 C CNN
+	1    1800 3550
+	1    0    0    -1
+$EndComp

Commit message: cob_2x2 v1.1:
- Fix inverter footprint
- Increase size of 5V TVS diode to SOD-523
- Increase clearance for mounting holes by 1mm
- Make mounting holes evenly spaced
Parts:
- U6: footprint Package_SO:TSSOP-8_3x3mm_P0.65mm -> Package_SO:SSOP-8_2.95x2.8mm_P0.65mm
